File: transmitter_schema/transmitter_schema.kicad_sch (KiCad schematic)
At the start: 16 parts, among them SW1 SW_SPDT, SW2 SW_Push, U1 PIC16F18324-xSL, U2 NRF24L01, U3 LM2937xT

Commit message: Refactors schematics
Parts:
- added D1: LED, LED_THT:LED_D5.0mm, symbol Device:LED
- added Q1: 2N7000, Package_TO_SOT_THT:TO-92_Inline_Wide, symbol ME218_BaseLib:2N7000
- added R3: 470, Resistor_THT:R_Axial_DIN0204_L3.6mm_D1.6mm_P7.62mm_Horizontal, symbol Device:R
- added RV3: R_Potentiometer, Potentiometer_THT:Potentiometer_Bourns_3386P_Vertical, symbol Device:R_Potentiometer
- BT1: footprint RC_Car_footprints:BAT_BH9VPC -> Connector_PinSocket_2.54mm:PinSocket_1x02_P2.54mm_Vertical
- RV1, RV2: footprint (none) -> transmitter_footprints:TRIM_PT01-D115D-B502; Field-1 (none) -> Same Sky (Formerly CUI Devices); Mfn (none) -> Same Sky (Formerly CUI Devices); Mfn PN (none) -> PT01-D115D-B502; Supplier (none) -> DigiKey; Supplier PN (none) -> 2223-PT01-D115D-B502-ND
Connections:
- net +3.3V: now also R3.1, RV3.1
- net GND: now also RV1.S1, RV1.S2, RV2.S1, RV2.S2, Q1.1 (S), RV3.3
- net LIGHTS: now reaches PRG1.4 (PGData), U1.13 (RA0)
- net LIGHTS: now also Q1.2 (G)
- net STEER_TRIM: now reaches U1.3 (RA4)
- net STEER_TRIM: now also RV3.2
- new net: D1.1 (K), Q1.3 (D)
- new net: D1.2 (A), R3.2
Other:
- moved on the sheet: RV1
