File: schematics/receiver/receiver.kicad_sch (KiCad schematic)
At the start: 26 parts, among them M1 Servo, M2 Motor, Q1 2N7000, Q2 2N7000, SW1 SW_Nidec_CAS-120A1, U1 PIC16F18324-xSL, U2 LM2937xT, U3 NRF24L01_Breakout, U4 L9110H

Commit message: Update
Parts:
- removed C1, C2: 0.1u, Capacitor_THT:CP_Radial_D5.0mm_P2.50mm, symbol Device:C
- removed C4: 10u, Capacitor_THT:CP_Radial_D5.0mm_P2.50mm, symbol Device:C
- removed JP1, JP2: SolderJumper_2_Open, Jumper:SolderJumper-2_P1.3mm_Open_RoundedPad1.0x1.5mm, symbol Jumper:SolderJumper_2_Open
- removed U1: PIC16F18324-xSL, Package_DIP:DIP-14_W7.62mm, symbol MCU_Microchip_PIC16:PIC16F18324-xSL
- removed U2: LM2937xT, Package_TO_SOT_THT:TO-220-3_Horizontal_TabDown, symbol Regulator_Linear:LM2937xT
- added BZ1: Buzzer, receiver:XDCR_AT-1224-TWT-5V-2-R, symbol Device:Buzzer
- added C1, C2, C5: 0.1u, Capacitor_SMD:C_0402_1005Metric, symbol ME218_BaseLib:Cap
- added C10: 22u, Capacitor_Tantalum_SMD:CP_EIA-2012-15_AVX-P, symbol Device:C
- added C7: 10u, Capacitor_SMD:C_0402_1005Metric, symbol Device:C
- added C9: 10u, Capacitor_SMD:C_0805_2012Metric, symbol Device:C
- added D1, D4: LED, Connector_PinSocket_2.54mm:PinSocket_1x02_P2.54mm_Vertical, symbol Device:LED
- added J1: Program, Connector_PinSocket_2.54mm:PinSocket_1x05_P2.54mm_Vertical, symbol Connector:Conn_01x05_Pin
- added J2: Debug, Connector_PinSocket_2.54mm:PinSocket_1x03_P2.54mm_Vertical, symbol Connector:Conn_01x03_Pin
- added Q3, Q4, Q5: 2N7000, Package_TO_SOT_SMD:SOT-23, symbol ME218_BaseLib:2N7000
- added R1, R10, R11, R9: 10k, Resistor_SMD:R_0402_1005Metric, symbol Device:R
- added R12, R2, R7: 470, Resistor_SMD:R_0402_1005Metric, symbol Device:R
- added R3: 1k, Resistor_SMD:R_0402_1005Metric, symbol Device:R
- added SW2: ~{MCLR}, pcb_radio:SW_1825910-6-4, symbol Switch:SW_Push
- added U5: PIC32MX170F256B, receiver:SSOP28_MC_MCH, symbol ME218_BaseLib:PIC32MX170F256B
- added U6: AMS1117-3.3, Package_TO_SOT_SMD:SOT-223-3_TabPin2, symbol Regulator_Linear:AMS1117-3.3
- C3: footprint Capacitor_THT:CP_Radial_D5.0mm_P2.50mm -> receiver:U2-K_NCH; Mfn KEMET -> Nichicon; Mfn PN ESY227M035AH1AA -> UWT1C221MCL1GS; Supplier PN 399-6122-ND -> 493-2179-2-ND
- D2, D3: footprint LED_THT:LED_D5.0mm -> Connector_PinSocket_2.54mm:PinSocket_1x02_P2.54mm_Vertical
- Q1, Q2: footprint Package_TO_SOT_THT:TO-92_Inline_Wide -> Package_TO_SOT_SMD:SOT-23; Mfn Diotec Semiconductor -> Toshiba Semiconductor and Storage; Mfn PN 2N7000 -> T2N7002AK,LM; Supplier PN 4878-2N7000CT-ND -> T2N7002AKLMTR-ND
- R4, R5: footprint Resistor_THT:R_Axial_DIN0204_L3.6mm_D1.6mm_P7.62mm_Horizontal -> Resistor_SMD:R_0402_1005Metric; Mfn Stackpole Electronics Inc -> YAGEO; Mfn PN CF14JT470R -> RC0402JR-07470RL; Supplier PN CF14JT470RTR-ND -> 311-470JRTR-ND
- R6: footprint Resistor_THT:R_Axial_DIN0204_L3.6mm_D1.6mm_P7.62mm_Horizontal -> Resistor_SMD:R_0402_1005Metric; Mfn Stackpole Electronics Inc -> YAGEO; Mfn PN CF14JT10K0 -> RC0402JR-0710KL; Supplier PN CF14JT10K0TR-ND -> 311-10KJRTR-ND
- R8: footprint Resistor_THT:R_Axial_DIN0204_L3.6mm_D1.6mm_P7.62mm_Horizontal -> Resistor_SMD:R_0402_1005Metric; Mfn Stackpole Electronics Inc -> YAGEO; Mfn PN CF14JT10K0 -> RC0402JR-0710KL; Supplier PN (none) -> 311-10KJRTR-ND
- SW1: value SW_Nidec_CAS-120A1 -> Power
Connections:
- net LIGHTS is gone; now on net GND: Q1.2 (S), Q2.2 (S), R6.1
- net PWM5.1 is gone; now on an unnamed net: U4.4 (OB)
- net +3.3V: now also C1.2, C10.1, C5.2, J1.2 (Pin_2), R1.2, R12.1, R2.1, R7.1, U5.13 (Vdd), U5.28 (AVdd), U6.2 (VO)
- net +9V: now also C9.1, U6.3 (VI)
- net CE: now also U5.26 (RB15)
- net CSN: now also U5.23 (RB12)
- net GND: now also R8.1, C1.1, C10.2, C2.1, C5.1, C7.2, C9.2, J1.3 (Pin_3), J2.3 (Pin_3), Q3.2 (S), Q4.2 (S), Q5.2 (S), R10.1, R11.1, R9.1, SW2.3, SW2.4, U5.19 (Vss), U5.27 (AVss), U5.8 (Vss), U6.1 (GND); no longer Q1.1 (S), Q2.1 (S), R6.2, R8.2
- net IRQ: now also U5.21 (PGEC2/5VT/RB10)
- net MISO: now also U5.22 (RB11)
- net MOSI: now also U5.24 (RB13)
- net PWM5: now also U4.7 (IB), U5.14 (PGED3/5VT/RB5); no longer U4.1 (OA)
- net PWM6: now also U5.12 (RA4)
- net SCK: now also U5.25 (RB14)
- net at D3.1 (K): now also Q3.3 (D); no longer Q2.3 (D)
- net at BT1.1 (+): now also SW1.2 (B)
- net at M2.1 (+): now also U4.1 (OA); no longer U4.7 (IB)
- net at M2.2 (-): no longer U4.6 (IA)
- new net: C2.2, R1.1, R3.2, SW2.1, SW2.2
- new net: C7.1, U5.20 (Vcap)
- new net: D1.2 (A), R2.2
- new net: D1.1 (K), Q2.3 (D)
- new net: D4.2 (A), R7.2
- new net: D4.1 (K), Q4.3 (D)
- new net: BZ1.2 (-), Q5.3 (D)
- new net: BZ1.1 (+), R12.2
- new net BL_LIGHTS: Q3.1 (G), R9.2, U5.18 (PGED2/5VT/RB9)
- new net BR_LIGHTS: Q4.1 (G), R10.2, U5.17 (5VT/RB8)
- new net FL_LIGHTS: Q1.1 (G), R6.2, U5.2 (RA0)
- new net FR_LIGHTS: Q2.1 (G), R8.2, U5.3 (RA1)
- new net HORN: Q5.1 (G), R11.2, U5.10 (RA3)
- new net PGClk: J1.5 (Pin_5), U5.5 (PGEC1/RB1)
- new net PGData: J1.4 (Pin_4), U5.4 (PGED1/RB0)
- new net PWM4: U4.6 (IA), U5.11 (RB4)
- new net RXD: J2.2 (Pin_2), U5.16 (5VT/RB7)
- new net TXD: J2.1 (Pin_1), U5.15 (PGEC3/5VT/RB6)
- new net ~{MCLR}: J1.1 (Pin_1), R3.1, U5.1 (~{MCLR})
- no-connect marks 1 -> 4
Other:
- note added: "MCU"
- note added: "Program and Debug"
- note added: "Reset Buttons"
- note removed: "PIC16LF18326"
- moved on the sheet: D2, Q1, R4
