File: schematics/receiver/receiver.kicad_sch (KiCad schematic)
At the start: 44 parts, among them J1 Program, J2 Debug, M1 Servo, M2 Motor, Q1 2N7000, Q2 2N7000, Q3 2N7000, Q4 2N7000, Q5 2N7000, SW1 Power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

Commit message: Update
Parts:
- added D5: LED, LED_SMD:LED_0402_1005Metric, symbol Device:LED
- added R13: 470, Resistor_SMD:R_0402_1005Metric, symbol Device:R
Connections:
- net +3.3V: now also R13.1
- net BL_LIGHTS: now also U5.10 (RA3); no longer U5.18 (PGED2/5VT/RB9)
- net GND: now also D5.1 (K)
- net HORN: now also U5.9 (RA2); no longer U5.10 (RA3)
- new net: D5.2 (A), R13.2
Other:
- moved on the sheet: BT1

Commit message: Update
Parts:
- removed BZ1: Buzzer, receiver:XDCR_AT-1224-TWT-5V-2-R, symbol Device:Buzzer
- added D6: LED, LED_SMD:LED_0402_1005Metric, symbol Device:LED
Connections:
- net +9V: now also SW1.2 (B); no longer SW1.3 (A)
- net GND: now also SW1.1 (C)
- net at BT1.1 (+): now also SW1.3 (A); no longer SW1.2 (B)
- net at Q5.3 (D): now also D6.1 (K)
- net at R12.2: now also D6.2 (A)
- net HORN renamed LED
- no-connect marks 4 -> 3
Other:
- note added: "PIC32MX170F256"
- note removed: "MCU"
- moved on the sheet: BT1, C1, C10, C2, C5, C7, C9, D3, D4, D5, Q3, Q4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

Commit message: UPdate
Other:
- note added: "Front Lights"
- note added: "Rear Lights"
- note added: "Status LED"
- note removed: "Lights"
- moved on the sheet: C2, D1, D2, D3, D4, D6, J1, J2, Q1, Q2, Q3, Q4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
