File: schematics/transmitter/transmitter.kicad_pcb (KiCad board)
At the start: 4 copper layers, 38 x 72.6 mm, 24 parts, among them Q1 2N7000, SW1 SW_Nidec_CAS-120A1, U1 PIC16F18324-xSL, U2 NRF24L01_Breakout, U3 LM2937xT

Commit message: Update
Parts:
- removed C4: 220u, Capacitor_THT:CP_Radial_D5.0mm_P2.50mm
- removed JP1, JP2: SolderJumper_2_Open, Jumper:SolderJumper-2_P1.3mm_Open_RoundedPad1.0x1.5mm
- removed Q1: 2N7000, Package_TO_SOT_THT:TO-92_Inline_Wide
- removed R2: 470, Resistor_THT:R_Axial_DIN0204_L3.6mm_D1.6mm_P7.62mm_Horizontal
- removed U1: PIC16F18324-xSL, Package_DIP:DIP-14_W7.62mm
- added C2: 0.1u, Capacitor_SMD:C_0402_1005Metric, F.Cu at (94.5, 81.6)
- added C6: 0.1u, Capacitor_SMD:C_0402_1005Metric, F.Cu at (83.7, 88.9)
- added C7: 10u, Capacitor_SMD:C_0402_1005Metric, F.Cu at (83.5, 83.2)
- added C8: 0.1u, Capacitor_SMD:C_0402_1005Metric, F.Cu at (89.5, 93.5)
- added J1: Program, Connector_PinSocket_2.54mm:PinSocket_1x05_P2.54mm_Vertical, F.Cu at (108.6, 73.0)
- added J2: Debug, Connector_PinSocket_2.54mm:PinSocket_1x03_P2.54mm_Vertical, F.Cu at (82.9, 72.4)
- added Q2: 2N7000, Package_TO_SOT_SMD:SOT-23, F.Cu at (105.4, 103.4)
- added R3: 10k, Resistor_SMD:R_0402_1005Metric, F.Cu at (87.1, 93.5)
- added R4: 1k, Resistor_SMD:R_0402_1005Metric, F.Cu at (91.9, 93.5)
- added RV4: Trim Pot, Potentiometer_THT:Potentiometer_Bourns_3386P_Vertical, F.Cu at (76.7, 61.7)
- added SW2: ~{MCLR}, pcb_radio:SW_1825910-6-4, F.Cu at (89.5, 97.7)
- added U4: PIC32MX170F256B, receiver:SSOP28_MC_MCH, F.Cu at (89.1, 84.7)
- BT1: value 9V Battery -> Battery_Cell
- C1: value 0.1u -> 10u; footprint Capacitor_THT:CP_Radial_D5.0mm_P2.50mm -> Capacitor_SMD:C_0805_2012Metric
- C3: value 0.1u -> 220u; footprint Capacitor_THT:CP_Radial_D5.0mm_P2.50mm -> receiver:U2-K_NCH
- C5: value 10u -> 22u; footprint Capacitor_THT:CP_Radial_D5.0mm_P2.50mm -> Capacitor_Tantalum_SMD:CP_EIA-2012-15_AVX-P
- D1, D2: footprint LED_THT:LED_D5.0mm -> LED_SMD:LED_0402_1005Metric
- R1, R5: footprint Resistor_THT:R_Axial_DIN0204_L3.6mm_D1.6mm_P7.62mm_Horizontal -> Resistor_SMD:R_0402_1005Metric
- R6: value 10k -> 470; footprint Resistor_THT:R_Axial_DIN0204_L3.6mm_D1.6mm_P7.62mm_Horizontal -> Resistor_SMD:R_0402_1005Metric
- RV1, RV2: value R_Potentiometer -> Control Pot
- RV3: value R_Potentiometer -> Trim Pot
- SW1: value SW_Nidec_CAS-120A1 -> Power
- U3: value LM2937xT -> AMS1117-3.3; footprint Package_TO_SOT_THT:TO-220-3_Horizontal_TabDown -> Package_TO_SOT_SMD:SOT-223-3_TabPin2
- moved R5 28.0 mm to (102.6, 107.5), turned to 180 degrees
- moved R1 23.3 mm to (98.2, 115.2), turned to 0 degrees
- moved D1 22.3 mm to (98.2, 112.6), turned to 0 degrees
- moved C3 14.0 mm to (77.8, 94.9), turned to 0 degrees
- moved BT1 9.00 mm to (91.5, 119.8)
- moved R6 8.18 mm to (105.0, 107.5)
- moved RV3 8.04 mm to (102.2, 61.7)
- moved U3 7.40 mm to (89.2, 112.8)
- moved C5 7.24 mm to (94.9, 113.7), turned to -90 degrees
- moved SW1 6.83 mm to (78.2, 116.2), turned to 180 degrees
- moved D2 4.16 mm to (107.4, 107.5), turned to 180 degrees
- moved C1 1.15 mm to (83.5, 114.2), turned to 90 degrees
Connections:
- D1 pad 1: Net-(D1-K) -> GND
- D2 pad 2: +3.3V -> Net-(D2-A)
- R5 pad 1: Net-(U1-RA5) -> GND
- R5 pad 2: +3.3V -> LED
- R6 pad 1: LED -> +3.3V
- R6 pad 2: GND -> Net-(D2-A)
- RV3 pad 2: TRIM -> STEER_TRIM
- SW1 pad 1: Net-(JP2-B) -> unconnected-(SW1-C-Pad1)
- SW1 pad 2: Net-(JP1-B) -> Net-(BT1-+)
- U3 pad 1: +9V -> GND
- U3 pad 2: GND -> +3.3V
- U3 pad 3: +3.3V -> +9V
Routing:
- net SPEED_TRIM: track 0.00 -> 29.6 mm
- net TRIM: track 28.4 -> 0.00 mm
- net ~{MCLR}: track 0.00 -> 27.9 mm
- net STEER_TRIM: track 0.00 -> 25.3 mm
- net GND: track 5.92 -> 24.2 mm, vias 0 -> 11
- net PGData: track 0.00 -> 18.0 mm
- net PGClk: track 0.00 -> 16.3 mm
- net +3.3V: track 11.3 -> 25.4 mm, vias 0 -> 6
- net Net-(C8-Pad2): track 0.00 -> 12.9 mm
- net Net-(U1-RA5): track 12.7 -> 0.00 mm
- net Net-(BT1-+): track 10.3 -> 0.00 mm
- net TXD: track 0.00 -> 9.16 mm
- net CSN: track 20.2 -> 11.2 mm, vias 0 -> 1
- net MOSI: track 20.8 -> 12.5 mm
- net +9V: track 17.6 -> 9.44 mm
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
Commit message: Update
Parts:
- moved SW1 5.13 mm to (78.2, 111.1), turned to 0 degrees
Connections:
- SW1 pad 1: unconnected-(SW1-C-Pad1) -> GND
- SW1 pad 2: Net-(BT1-+) -> +9V
- SW1 pad 3: +9V -> Net-(BT1-+)
Routing:
- net Net-(BT1-+): track 0.00 -> 14.8 mm
- net +9V: track 9.44 -> 8.47 mm

Commit message: UPdate
Other:
- board text added: "1"
- board text added: "5"
- board text added: "GND"
- board text added: "RX"
- board text added: "TX"
Changed lines of the file:
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@@
 		(tags "Through hole socket strip THT 1x03 2.54mm single row")
 		(property "Reference" "SW1"
-			(at 0 -2.77 360)
+			(at 0 -2.77 0)
 			(layer "F.SilkS")
 			(hide yes)
@@
 		)
 		(property "Value" "Power"
-			(at 0 7.85 360)
+			(at 0 7.85 0)
 			(layer "F.SilkS")
 			(effects
@@
 		)
 		(property "Value" "Program"
-			(at -2.27 8.58 0)
+			(at -2.495 5.18 0)
 			(layer "F.SilkS")
 			(effects
@@
 		(layer "Edge.Cuts")
 	)
+	(gr_text "5"
+		(at 97.86 71.02 0)
+		(layer "F.SilkS")
+		(effects
+			(font
+				(size 1 1)
+				(thickness 0.2)
+				(bold yes)
+			)
+			(justify left bottom)
+		)
+	)
+	(gr_text "TX"
+		(at 84.62 73.06 0)
+		(layer "F.SilkS")
+		(effects
+			(font
+				(size 1 1)
+				(thickness 0.2)
+				(bold yes)
+			)
+			(justify left bottom)
+		)
+	)
+	(gr_text "GND"
+		(at 84.5 78.06 0)
+		(layer "F.SilkS")
+		(effects
+			(font
+				(size 1 1)
+				(thickness 0.2)
+				(bold yes)
+			)
+			(justify left bottom)
+		)
+	)
+	(gr_text "RX"
+		(at 84.49 75.42 0)
+		(layer "F.SilkS")
+		(effects
+			(font
+				(size 1 1)
+				(thickness 0.2)
+				(bold yes)
+			)
+			(justify left bottom)
+		)
+	)
+	(gr_text "1"
+		(at 108.05 71.08 0)
+		(layer "F.SilkS")
+		(effects
+			(font
+				(size 1 1)
+				(thickness 0.2)
+				(bold yes)
+			)
+			(justify left bottom)
+		)
+	)
 	(segment
